File: stm32f091-ref_Lauren/_autosave-stm32f091.sch (KiCad schematic (older format))
At the start: 26 parts, among them J1 Conn_01x30_Male, J2 Conn_01x30_Male, J3 Conn_02x05_Odd_Even, SW1 SW_Push, U1 LD1117S33TR_SOT223, U2 STM32F091RCTx

Commit message: drew kicad schematic for keypad and speaker circuit
Parts:
- added C11, C13: 10uF, Capacitor_SMD:C_0805_2012Metric_Pad1.15x1.40mm_HandSolder, symbol Device:C
- added C12, C15: 0.1uF, Capacitor_SMD:C_0805_2012Metric_Pad1.15x1.40mm_HandSolder, symbol Device:C
- added C14: 220uF, Capacitor_SMD:C_0805_2012Metric_Pad1.15x1.40mm_HandSolder, symbol Device:C
- added C?: C_Polarized, symbol Device:C_Polarized
- added J?: Conn_01x02_Female, symbol Connector:Conn_01x02_Female
- added J?: Conn_01x08_Female, symbol Connector:Conn_01x08_Female
- added R10, R11, R12, R6, R7, R8, R9: 1K, Resistor_SMD:R_0805_2012Metric_Pad1.15x1.40mm_HandSolder, symbol Device:R_US
- added R13: 1.2K, Resistor_SMD:R_0805_2012Metric_Pad1.15x1.40mm_HandSolder, symbol Device:R_US
- added R14: 10, Resistor_SMD:R_0805_2012Metric_Pad1.15x1.40mm_HandSolder, symbol Device:R_US
- added RV1: R_Potentiometer_US, symbol Device:R_Potentiometer_US
- added U?: LM386, symbol Amplifier_Audio:LM386
- renumbered C11 to C10
Connections:
- wire segments 165 -> 225
Other:
- moved on the sheet: R13
