File: stm32f091-ref_Lauren/stm32f091.kicad_pcb (KiCad board)
At the start: 4 copper layers, 20.3 x 85.1 mm, 46 parts, among them J1 Conn_01x30_Male, J2 Conn_01x30_Male, J3 Conn_02x05_Odd_Even, J4 Conn_02x03_Odd_Even, J5 Conn_02x03_Odd_Even, SW1 SW_Push, SW2 SW_Push, SW3 SW_Push, U1 LD1117S33TR_SOT223, U2 STM32F091RCTx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

Commit message: drew kicad schematic for keypad and speaker circuit
Routing:
- added copper zone on In2.Cu, net +3V0
- added copper zone on In1.Cu, net GND
- removed copper zone on Power.Cu, net +3V0
- removed copper zone on Ground.Cu, net GND
Other:
- net class Default removed
