File: stm32f091-ref_Master_separate_power_supply/stm32f091.kicad_sch (KiCad schematic)
At the start: 62 parts, among them J1 Conn_02x05_Odd_Even, J2 Conn_01x08_Female, J3 Conn_01x02_Female, J4 Conn_01x09_Female, SW1 SW_Push, U1 LD1117S33TR_SOT223, U2 LM324, U3 STM32F091RCTx, U4 LM386

Commit message: changed r's and c's to SM in condensed PCB design
Parts:
- C19: renamed from C20; value (none) -> .1uF
- J2: renamed from J4; footprint (none) -> local_models:J3
- LD1, LD2: footprint (none) -> LED_THT:LED_D2.0mm_W4.8mm_H2.5mm_FlatTop
- RV1, RV2: footprint Potentiometer_THT:Potentiometer_Omeg_PC16BU_Vertical -> local_models:potentiometer
- U2: footprint (none) -> local_models:U2
- U4: footprint (none) -> local_models:U4
- renumbered C21 to C20, C19 to C21, J2 to J3, J3 to J4, R14 to R13, R15 to R14, R16 to R15, R17 to R16, R18 to R17, R19 to R18, R20 to R19, R21 to R20, R13 to R21
