File: stm32f091-ref_Master/stm32f091_project_condensed.kicad_pcb (KiCad board)
At the start: 4 copper layers, 56 x 42.7 mm, 62 parts, among them J1 Conn_02x05_Odd_Even, J2 Conn_01x09_Female, J3 Conn_01x08_Female, J4 Conn_01x02_Female, SW1 SW_Push, U1 LD1117S33TR_SOT223, U2 LM324, U3 STM32F091RCTx, U4 LM386

Commit message: new pcb design
Parts:
- added R22: 10k, Resistor_SMD:R_0805_2012Metric_Pad1.20x1.40mm_HandSolder, F.Cu at (118.4, 130.0)
- added SW2: SW_Push, Button_Switch_SMD:SW_SPST_PTS645, F.Cu at (107.7, 130.7)
- C18: footprint Capacitor_SMD:C_0805_2012Metric_Pad1.18x1.45mm_HandSolder -> Capacitor_THT:CP_Radial_D10.0mm_P5.00mm
- moved D3 35.3 mm to (85.9, 140.1), turned to 90 degrees
- moved C18 26.9 mm to (131.8, 109.1)
- moved R8 7.05 mm to (111.8, 120.3)
- moved J4 5.04 mm to (93.0, 138.9)
- moved C20 1.96 mm to (140.0, 115.5)
- moved U1 1.93 mm to (93.5, 124.4)
- moved R5 1.74 mm to (113.6, 124.6)
- moved D1 1.68 mm to (111.3, 136.1)
- moved R1 1.54 mm to (109.0, 141.1)
- moved C7 1.53 mm to (105.4, 141.1)
- moved R6 1.49 mm to (110.0, 124.6)
- moved R12 1.45 mm to (114.1, 114.7)
- moved J3 1.34 mm to (135.1, 101.0)
- moved R3 1.24 mm to (106.4, 124.6)
- moved R13 1.03 mm to (124.7, 108.6)
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