File: stm32f091-ref_Master/_autosave-stm32f091_project_condensed.kicad2_pcb.kicad_pcb3.kicad_pcb (KiCad board)
At the start: 4 copper layers, 68.8 x 53.3 mm, 64 parts, among them J1 Conn_02x05_Odd_Even, J2 Conn_01x09_Female, J3 Conn_01x08_Female, J4 Conn_01x02_Female, SW1 SW_Push, SW2 SW_Push, U1 LD1117S33TR_SOT223, U2 LM324, U3 STM32F091RCTx, U4 LM386

Commit message: new pcb after diode and 324 changes
Routing:
- net +3V0: track 161.4 -> 171.1 mm, vias 6 -> 7
Changed lines of the file:
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@@
     )
   )
-  (gr_circle (center 127.973659 119.55876) (end 128.481659 119.81276) (layer "F.SilkS") (width 0.12) (fill none))
+  (gr_circle (center 130.69 117.612039) (end 131.257961 117.612039) (layer "F.SilkS") (width 0.4) (fill none))
   (gr_rect (start 79.01162 152.57876) (end 147.84562 99.23876) (layer "Edge.Cuts") (width 0.05) (fill none))
   (gr_text "PillCB - Team 16 (4/13/2022 - V01)\nJaideep Damle, Lauren Gunter, \nNidhi Kunigal, Elizabeth McNaughton" (at 111.76 116.84) (layer "B.SilkS")
@@
   (segment (start 120.893939 126.350241) (end 121.487913 125.756267) (width 0.25) (layer "F.Cu") (net 11))
   (segment (start 106.426 120.65) (end 106.426 119.25314) (width 0.25) (layer "F.Cu") (net 11))
+  (segment (start 85.86962 140.13276) (end 90.55686 144.82) (width 0.25) (layer "F.Cu") (net 11))
   (segment (start 120.41362 116.51076) (end 119.65162 116.51076) (width 0.25) (layer "F.Cu") (net 11))
   (segment (start 120.186833 113.728385) (end 119.38 112.921552) (width 0.25) (layer "F.Cu") (net 11))
@@
   (segment (start 119.38 112.921552) (end 119.38 111.95552) (width 0.25) (layer "F.Cu") (net 11))
   (segment (start 106.22362 119.05076) (end 106.22362 115.05276) (width 0.25) (layer "F.Cu") (net 11))
+  (segment (start 90.55686 144.82) (end 111.76 144.82) (width 0.25) (layer "F.Cu") (net 11))
   (segment (start 128.919601 118.324579) (end 128.919601 121.046941) (width 0.25) (layer "F.Cu") (net 11))
   (segment (start 122.361669 118.458809) (end 120.41362 116.51076) (width 0.25) (layer "F.Cu") (net 11))
@@
   (via (at 106.426 120.65) (size 0.8) (drill 0.4) (layers "F.Cu" "B.Cu") (net 11))
   (via (at 112.53374 126.22626) (size 0.8) (drill 0.4) (layers "F.Cu" "B.Cu") (net 11))
+  (via (at 111.76 144.82) (size 0.8) (drill 0.4) (layers "F.Cu" "B.Cu") (net 11))
   (via (at 118.579671 113.392425) (size 0.8) (drill 0.4) (layers "F.Cu" "B.Cu") (net 11))
   (via (at 121.158 127.254) (size 0.8) (drill 0.4) (layers "F.Cu" "B.Cu") (net 11))
   (via (at 122.361669 118.938331) (size 0.8) (drill 0.4) (layers "F.Cu" "B.Cu") (net 11))
-  (segment (start 111.26962 136.06876) (end 108.684131 138.654249) (width 0.25) (layer "In1.Cu") (net 11))
-  (segment (start 108.684131 138.654249) (end 87.348131 138.654249) (width 0.25) (layer "In1.Cu") (net 11))
-  (segment (start 87.348131 138.654249) (end 85.86962 140.13276) (width 0.25) (layer "In1.Cu") (net 11))
   (segment (start 118.579671 114.994545) (end 121.328386 117.74326) (width 0.25) (layer "In2.Cu") (net 11))
   (segment (start 121.328386 117.74326) (end 121.328386 117.905048) (width 0.25) (layer "In2.Cu") (net 11))
@@
   (segment (start 113.266497 124.744129) (end 111.580374 123.058006) (width 0.25) (layer "B.Cu") (net 11))
   (segment (start 109.172368 120.65) (end 106.426 120.65) (width 0.25) (layer "B.Cu") (net 11))
+  (segment (start 111.76 144.82) (end 111.26962 144.32962) (width 0.25) (layer "B.Cu") (net 11))
+  (segment (start 111.26962 144.32962) (end 111.26962 136.06876) (width 0.25) (layer "B.Cu") (net 11))
   (segment (start 116.977874 131.942126) (end 116.977874 128.674383) (width 0.25) (layer "B.Cu") (net 11))
   (segment (start 111.580374 123.058006) (end 109.172368 120.65) (width 0.25) (layer "B.Cu") (net 11))
