File: stm32f091-ref_Master/stm32f091_project_condensed_v02_afterchange.kicad_pcb (KiCad board)
At the start: 2 copper layers, 62.3 x 65 mm, 68 parts, among them J1 Conn_02x05_Odd_Even, J2 Conn_01x09_Female, J3 Conn_01x08_Female, J4 Conn_01x02_Female, SW1 SW_Push, SW2 SW_Push, U1 LD1117S33TR_SOT223, U2 LM324, U3 STM32F091RCTx, U4 LM386

Commit message: changed silkscreen to not overlap (no warnings) and created gerber files (plot_v02_approved)
Parts:
- moved R13 3.71 mm to (115.8, 100.8), turned to 180 degrees
- moved LS1 1.55 mm to (140.8, 139.4)
- moved R5 1.23 mm to (114.8, 127.4)
- moved C14 1.16 mm to (137.0, 138.7)
- moved R8 1.11 mm to (116.8, 127.2)
- moved C7 0.81 mm to (111.5, 127.0)
- moved C12 0.71 mm to (118.8, 127.7)
- moved C15 0.66 mm to (133.7, 138.7)
- moved C13 0.48 mm to (127.6, 138.6)
- moved R3 0.33 mm to (109.3, 127.7)
- moved R6 0.27 mm to (112.0, 123.1)
- moved R9 0.12 mm to (130.6, 138.7)
Routing:
- net GND: track 147.3 -> 137.8 mm
- net 3.3V: track 234.3 -> 228.6 mm
- net Net-(R7-Pad2): track 30.5 -> 25.3 mm
- net Net-(J3-Pad1): track 8.42 -> 12.7 mm
- net 5.5V: track 191.0 -> 193.1 mm
- net /PC6: track 33.6 -> 31.5 mm
- net /PC7: track 30.9 -> 29.0 mm
- net Net-(C15-Pad1): track 1.92 -> 3.02 mm
- net Net-(R5-Pad2): track 12.5 -> 11.5 mm, vias 1 -> 0
- net Net-(RV2-Pad2): track 10.0 -> 11.0 mm
- net /PC5: track 20.3 -> 21.2 mm
- net /PA4: track 33.9 -> 33.1 mm
- net Net-(C7-Pad1): track 35.0 -> 35.8 mm
- net Net-(C18-Pad2): track 46.1 -> 45.5 mm
